Commit message: minor corrections

File: sagan_description/model/Sagan.xacro.urdf (robot description, URDF)
Before this commit: robot Sagan, 18 links, 17 joints
Joints:
- joint LF_wheel_joint: axis 0 0 1 -> 0 0 -1
- joint LR_wheel_joint: axis 0 0 1 -> 0 0 -1
- joint RF_wheel_joint: axis 0 0 -1 -> 0 0 1
- joint RR_wheel_joint: axis 0 0 -1 -> 0 0 1
- joint base_footprint_joint: origin xyz=0 0 0.017 rpy=-1.5708 0 0 -> xyz=0 0 0.017 rpy=-1.5708 0 3.1415

Commit message: nav2 and slam package added

File: sagan_description/model/Sagan.xacro.urdf (robot description, URDF)
Before this commit: robot Sagan, 18 links, 17 joints
Links:
- removed link efk_reference
- removed link gz_reference
- removed link noise_odometry
- removed link odom
- removed link odom_gz_link
- added link lidar_frame
- link imu_link: mass 0 -> None
Joints:
- removed joint odom_efk_joint
- removed joint odom_gz_joint
- removed joint odom_gz_reference_joint
- removed joint odom_noise_joint
- removed joint odom_to_base_footprint
- added joint lidar_frame_joint: type fixed, parent base_link, child lidar_frame, origin xyz=0 -0.1 0 rpy=-1.5708 0 3.1415, axis 0 0 0
- joint base_footprint_joint: origin xyz=0 0 0.017 rpy=-1.5708 0 3.1415 -> xyz=0 0 0.2 rpy=-1.5708 0 3.1415

Commit message: mensagem

File: sagan_description/model/Sagan.xacro.urdf (robot description, URDF)
Before this commit: robot Sagan, 14 links, 13 joints
Links:
- added link camera_link
- link LF_stering_arm: geometry visual mesh filename=package://sagan_description/model/meshes/LF_stering_arm.STL
- link LF_wheel: geometry collision sphere radius=0.06; visual mesh filename=package://sagan_description/model/meshes/LF_wheel.STL
- link LR_stering_arm: geometry visual mesh filename=package://sagan_description/model/meshes/LR_stering_arm.STL
- link LR_wheel: geometry collision sphere radius=0.06; visual mesh filename=package://sagan_description/model/meshes/LR_wheel.STL
- link Left_arm: geometry collision mesh filename=package://sagan_description/model/meshes/Left_arm.STL; visual mesh filename=package://sagan_description/model/meshes/Left_arm.STL
- link RF_stering_arm: geometry visual mesh filename=package://sagan_description/model/meshes/RF_stering_arm.STL
- link RF_wheel: geometry collision sphere radius=0.06; visual mesh filename=package://sagan_description/model/meshes/RF_wheel.STL
- link RR_stering_arm: geometry visual mesh filename=package://sagan_description/model/meshes/RR_stering_arm.STL
- link RR_wheel: geometry collision sphere radius=0.06; visual mesh filename=package://sagan_description/model/meshes/RR_wheel.STL
- link Right_arm: geometry collision mesh filename=package://sagan_description/model/meshes/Right_arm.STL; visual mesh filename=package://sagan_description/model/meshes/Right_arm.STL
- link base_link: geometry collision mesh filename=package://sagan_description/model/meshes/base_link.STL; visual mesh filename=package://sagan_description/model/meshes/base_link.STL
Joints:
- added joint camera_joint: type fixed, parent base_link, child camera_link, origin xyz=-0.2 0.0 0.0 rpy=-1.5708 0 -3.1415
- joint Left_arm_joint: axis 0 0 0 -> (none)
- joint Right_arm_joint: axis 0 0 0 -> (none)
- joint imu_joint: axis 0 0 0 -> (none)
- joint lidar_frame_joint: axis 0 0 0 -> (none)

Commit message: imu params modified

File: sagan_description/model/Sagan.xacro.urdf (robot description, URDF)
Before this commit: robot Sagan, 15 links, 14 joints
Joints:
- joint lidar_frame_joint: origin xyz=0 -0.1 0 rpy=-1.5708 0 3.1415 -> xyz=0 -0.1 0 rpy=-1.5708 -3.1415  3.1415
